File: Hardware/Qwiic_TMP117.brd (EAGLE design)
At the start: 22.9 x 24.1 mm, 43 parts, among them J1 PTH, U2 TMP117

Commit message: Updated PCB
PCB updated to meet the jlcpcb specs with new milling width
Parts:
- moved C1 0.63 mm to (8.26, 7.62)
- moved R3 0.63 mm to (14.6, 7.62)
Routing:
- net 3.3V: track 66.3 -> 69.2 mm
- net SDA: track 49.5 -> 50.8 mm
- net GND: track 4.15 -> 5.17 mm
- net ADD0: track 19.7 -> 18.8 mm
- net SCL: track 48.1 -> 47.3 mm
- net !INT: track 17.9 -> 18.5 mm
- net N$4: track 4.27 -> 3.66 mm
Other:
- outline, holes or cut-outs redrawn
